File: motorBoard.sch (EAGLE design)
At the start: 58 parts

Commit message: Added decoupling caps, schematic tweaks, layout, mid routing
Running out of space around PSoC, so I need to rework my component layout.
Parts:
- removed LED8: (no value), eagle-ltspice:LED_E
- removed RA, RB, RC, RD: 4.7k, eagle-ltspice:RR1206
- removed U$10: SMD4SWSMD4SW, HuskyRobotics2017-18:SMD4SWSMD4SW
- added C1, C6: 1uF, eagle-ltspice:CC1206
- added C10, C11, C12, C13, C2, C3, C7, C8, C9: 0.1uF, eagle-ltspice:CC1206
- added C4, C5: 10uF, eagle-ltspice:CC1206
- added CAN: 22-23-2021, con-molex:22-23-2021
- added R10, R11, R12, R9: 4.7k, eagle-ltspice:RR1206
- added R13: 120, eagle-ltspice:RR1206
- added SHIFT_EN: SMD4SWSMD4SW, HuskyRobotics2017-18:SMD4SWSMD4SW
- added TCAN: TCAN332TCAN332, HuskyRobotics2017-18:TCAN332TCAN332
- added U$2: PUSH_BUTTON, HuskyRobotics2017-18:PUSH_BUTTON
- R1: value (none) -> 1.2k
- R2: value (none) -> 150
- R3, R4, R5, R6, R7: value (none) -> 100
- R8: value (none) -> 4.7k
- U$1: value TCAN332TCAN332 -> OOPS_SPACE; device HuskyRobotics2017-18:TCAN332TCAN332 -> HuskyRobotics2017-18:OOPS_SPACE
- renumbered BASIC_HEADER to SWD, LED1 to 24V, LED2 to 5V, LED3 to 3.3V, LED4 to 4, LED5 to 5, LED6 to 6, LED7 to 7, OKI-78SR-3.3 to 3.3V_DC-DC, OKI-78SR-5 to 5V_DC-DC, OSCILLATOR_SG-646PCE to OSC, U$3 to FEEDBACK, U$6 to SHIFT3, U$7 to SHIFT2, U$8 to SHIFT1, U$9 to SHIFT4
Connections:
- removed net LED8: LED8.A, PSOC4200L.VBUS/P13.2
- removed net N$23: LED8.C, R8.2
- new net VCCD: C1.1, PSOC4200L.VCCD
- new net VREF: C6.2, PSOC4200L.P1.7/VREF
- new net XRES: C7.2, PSOC4200L.XRES, R12.2, U$2.P
- net +3V3: now also C13.2, C3.2, C4.2, C7.1, C8.2, SHIFT_EN.1A, SHIFT_EN.2A, SHIFT_EN.3A, SHIFT_EN.4A, TCAN.VCC, U$2.S; no longer POT1.1, POT2.1, POT3.1, POT4.1, PSOC4200L.VCCD, PSOC4200L.VDDD, U$1.VCC, U$10.1A, U$10.2A, U$10.3A, U$10.4A
- net +5V: now also C10.2, C11.2, C12.2, C2.2, C5.2, C9.2, POT1.1, POT2.1, POT3.1, POT4.1, PSOC4200L.VDDD
- net CANH: now also CAN-1.S, R13.2, TCAN.CANH; no longer U$1.CANH
- net CANL: now also CAN-2.S, R13.1, TCAN.CANL; no longer U$1.CANL
- net CANRX: now also TCAN.RXD; no longer U$1.RXD
- net CANTX: now also TCAN.TXD; no longer U$1.TXD
- net GNDA: now also C1.2, C10.1, C11.1, C12.1, C13.1, C2.1, C3.1, C4.1, C5.1, C6.1, C8.1, C9.1, R10.1, R11.1, R12.1, R9.1, TCAN.GND; no longer RA.1, RB.1, RC.1, RD.1, U$1.GND
- net LED4: now also PSOC4200L.VBUS/P13.2; no longer PSOC4200L.P1.7/VREF
- net LEVEL_SHIFT_EN1: now also R11.2, SHIFT_EN.1B; no longer RD.2, U$10.1B
- net LEVEL_SHIFT_EN2: now also R10.2, SHIFT_EN.2B; no longer RC.2, U$10.2B
- net LEVEL_SHIFT_EN3: now also R9.2, SHIFT_EN.3B; no longer RB.2, U$10.3B
- net LEVEL_SHIFT_EN4: now also R8.2, SHIFT_EN.4B; no longer RA.2, U$10.4B
Other:
- note added: "Do limit switches need debounce caps?"
- note added: "Power connector?"
- note added: "What's a typical debounce cap value?"
- moved on the sheet: R8

Commit message: Finished Board
Ready for Review
Parts:
- removed C3: 0.1uF, eagle-ltspice:CC1206
Connections:
- net +3V3: now also U$1.3V3-1, U$1.3V3-2, U$1.3V3-3; no longer C3.2
- net +5V: now also U$1.5V-1, U$1.5V-2, U$1.5V-3
- net GNDA: now also U$1.GND-1, U$1.GND-2, U$1.GND-3, U$1.GND-4, U$1.GND-5, U$1.GND-6; no longer C3.1
Other:
- note added: "Removed Cap 3 because oscx cap serves same location on board"

Commit message: Revert "Finished Board"
This reverts commit 761fd842cb1d32e6d861dcd06b5bacfd84886b14.
Parts:
- added C3: 0.1uF, eagle-ltspice:CC1206
Connections:
- net +3V3: now also C3.2; no longer U$1.3V3-1, U$1.3V3-2, U$1.3V3-3
- net +5V: no longer U$1.5V-1, U$1.5V-2, U$1.5V-3
- net GNDA: now also C3.1; no longer U$1.GND-1, U$1.GND-2, U$1.GND-3, U$1.GND-4, U$1.GND-5, U$1.GND-6
Other:
- note removed: "Removed Cap 3 because oscx cap serves same location on board"

Commit message: Fixed Git Issues
If this push works, this should be the end of the git-astrophe.
Parts:
- removed C3: 0.1uF, eagle-ltspice:CC1206
Connections:
- net +3V3: now also U$1.3V3-1, U$1.3V3-2, U$1.3V3-3; no longer C3.2
- net +5V: now also U$1.5V-1, U$1.5V-2, U$1.5V-3
- net GNDA: now also U$1.GND-1, U$1.GND-2, U$1.GND-3, U$1.GND-4, U$1.GND-5, U$1.GND-6; no longer C3.1
Other:
- note added: "Removed Cap 3 because oscx cap serves same location on board"
